File: keypad.kicad_sch (KiCad schematic)
At the start: 8 parts, among them J1 Capacitive touch buttons, SW1 SW_Push, SW2 SW_Push, SW3 SW_Push, U1 XIAO-ESP32-S3

Commit message: fixed pcb wiring sorry!!
Connections:
- net LED: now also U1.10 (D9/GPIO8); no longer U1.11 (D10/GPIO9)
- net SWITCH3: now also U1.9 (D8/GPIO7); no longer U1.10 (D9/GPIO8)
- net TOUCH7: now also U1.11 (D10/GPIO9); no longer U1.9 (D8/GPIO7)
Changed lines of the file:
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@@
 		)
 	)
-	(label "LED"
-		(at 81.28 60.96 0)
+	(label "TOUCH4"
+		(at 27.94 55.88 0)
 		(effects
 			(font
@@
 		)
 	)
-	(label "TOUCH4"
-		(at 27.94 55.88 0)
+	(label "TOUCH7"
+		(at 81.28 60.96 0)
 		(effects
 			(font
@@
 	(label "TOUCH2"
 		(at 31.75 106.68 0)
-		(effects
-			(font
-				(size 1.27 1.27)
-			)
-			(justify left bottom)
-		)
-	)
-	(label "SWITCH3"
-		(at 81.28 58.42 0)
 		(effects
 			(font
@@
 	(label "SWITCH2"
 		(at 132.08 114.3 0)
-		(effects
-			(font
-				(size 1.27 1.27)
-			)
-			(justify left bottom)
-		)
-	)
-	(label "TOUCH7"
-		(at 81.28 55.88 0)
 		(effects
 			(font
@@
 		)
 	)
+	(label "SWITCH3"
+		(at 81.28 55.88 0)
+		(effects
+			(font
+				(size 1.27 1.27)
+			)
+			(justify left bottom)
+		)
+	)
 	(label "TOUCH1"
 		(at 31.75 104.14 0)
 		(effects
 			(font
+				(size 1.27 1.27)
+			)
+			(justify left bottom)
+		)
+	)
+	(label "LED"
+		(at 81.28 58.42 0)
+		(effects
+			(font
